File: Board.sch (EAGLE design)
At the start: 56 parts, among them IC1 CP210X_USB_UART, T1 BC846, T2 BC846

Commit message: cleanup schematic
Parts:
- removed U$5: SPDT_GROUNDED, SparkFun-Electromechanical:SPDT_GROUNDED
- added S1: SPDT_GROUNDED, SparkFun-Electromechanical:SPDT_GROUNDED
- R1, R2: value (none) -> 470
- R16: value 220k -> 50k
- R17: value 100k -> 220k
- S4: value DOWN -> UP
- S5: value UP -> DOWN
Connections:
- net GND: now also S1G$2.1; no longer U$5G$2.1
- net N$17: now also S1G$1.S; no longer U$5G$1.S
- net V+: now also S1G$1.P; no longer U$5G$1.P
Other:
- moved on the sheet: C1, C2, C3, C4, C5, C6, J1, L1, LED1, LED2, LED3, MDL1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

Commit message: moved pins to new spi out and removed unused components
Parts:
- removed LED2: Charged, led:LEDSML0805
- removed LED3: (no value), led:LEDSML0805
- removed R1: 470, rcl:R-EU_R0603
- removed S5: DOWN, SparkFun-Electromechanical:SWITCH-MOMENTARY-2SMD-1101NE
- removed S6: LEFT, SparkFun-Electromechanical:SWITCH-MOMENTARY-2SMD-1101NE
- removed S7: RIGHT, SparkFun-Electromechanical:SWITCH-MOMENTARY-2SMD-1101NE
- removed SJ2: HW CS, SparkFun-Retired:SOLDERJUMPERNO
- removed SJ3: SW CS, SparkFun-Retired:SOLDERJUMPERNO
- added POWER: (no value), led:LEDSML0805
- added R20: 470, rcl:R-EU_R0603
- R15: value 470 -> 1k
- S2: value USER -> FLASH
- S3: value FLASH -> USER
- S4: value UP -> RIGHT
Connections:
- removed net GPIO10: MDL1.GPIO10, S7.1
- removed net GPIO12: MDL1.GPIO12, S5.1
- removed net GPIO13: MDL1.GPIO13, S4.1
- removed net GPIO14: MDL1.GPIO14, S6.1
- removed net N$11: MDL1.GPIO2, R9.2
- removed net N$20: MDL1.GPIO15, R12.2
- removed net N$23: MDL1.CS0, SJ2.2
- removed net N$25: MDL1.GPIO9, SJ3.2
- removed net N$9: LED2.A, R1.1
- new net GPIO2: MDL1.GPIO2, R20.1, R9.2
- new net N$29: R20.2, S4.2
- net CS: now also MDL1.GPIO15, R12.2; no longer SJ2.1, SJ3.1
- net GND: now also POWER.C, S4.1; no longer LED2.C, S4.2, S5.2, S6.2, S7.2
- net GPIO16: no longer LED3.C
- net MISO: now also MDL1.GPIO12; no longer MDL1.MISO
- net MOSI: now also MDL1.GPIO13; no longer MDL1.MOSI
- net N$10: no longer R1.2
- net N$21: now also S3.2; no longer S2.2
- net N$22: now also S2.2; no longer S3.2
- net N$24: now also POWER.A; no longer LED3.A
- net SCK: now also MDL1.GPIO14; no longer MDL1.SCLK
Other:
- moved on the sheet: C5, R15, R9, S2, S3, S4
